Commit message: urdfファイルの中身melodicからnoeticに修正

File: hsr_description/robots/hsrb4s.urdf (robot description, URDF)
Before this commit: robot hsrb, 45 links, 44 joints
Joints:
- joint arm_lift_joint: origin xyz=0.0 0.0 0.340 rpy=0.0 0.0 0.0 -> (none)
- joint base_imu_frame_joint: origin xyz=0.0005 0.1296 0.181 rpy=3.14159265359 0.0 0.0 -> (none)
- joint base_l_drive_wheel_joint: origin xyz=-0.11 0.133 0.04 rpy=0.0 0.0 0.0 -> (none)
- joint base_l_passive_wheel_x_frame_joint: origin xyz=0.1495                 0.055                 0.03 rpy=0.0 0.0 0.0 -> (none)
- joint base_r_drive_wheel_joint: origin xyz=-0.11 -0.133 0.04 rpy=0.0 0.0 0.0 -> (none)
- joint base_r_passive_wheel_x_frame_joint: origin xyz=0.1495                 -0.055                 0.03 rpy=0.0 0.0 0.0 -> (none)
- joint base_range_sensor_joint: origin xyz=0.1675 0.0 0.1844 rpy=0.0 0.0 0.0 -> (none)
- joint hand_camera_frame_joint: origin xyz=0.039 0.0 -0.0045 rpy=0.0 0.0 0.0 -> (none)
- joint hand_camera_gazebo_frame_joint: origin xyz=0 0 0 rpy=1.5707963268 -1.5707963268 0 -> xyz=0 0 0 rpy=1.570796326795 -1.570796326795 0
- joint hand_l_distal_joint: axis 1.0 0.0 0.0 -> (none)
- joint hand_l_finger_tip_frame_joint: origin xyz=0.01675 0.0193 0.0379 rpy=-1.5707963268 0.0 0.0 -> xyz=0.01675 0.0193 0.0379 rpy=-1.570796326795 0.0 0.0
- joint hand_l_finger_vacuum_frame_joint: origin xyz=0.00475 -0.011539 0.03322 rpy=0.785398163398 0.0 0.0 -> xyz=0.00475 -0.011539 0.03322 rpy=0.7853981633975 0.0 0.0
- joint hand_l_mimic_distal_joint: axis 1.0 0.0 0.0 -> (none); origin xyz=0.0 0.0 0.07 -> (none)
- joint hand_l_proximal_joint: axis 1.0 0.0 0.0 -> (none); origin xyz=-0.01675 -0.0245 -0.0175 rpy=0.0 0.0 0.0 -> (none)
- joint hand_l_spring_proximal_joint: axis 1.0 0.0 0.0 -> (none)
- joint hand_palm_joint: origin xyz=0.012 0.0 0.1405 rpy=0.0 0.0 3.14159265359 -> (none)
- joint hand_r_distal_joint: axis -1.0 0.0 0.0 -> (none)
- joint hand_r_finger_tip_frame_joint: origin xyz=0.01675 -0.0193 0.0379 rpy=1.5707963268 0.0 0.0 -> xyz=0.01675 -0.0193 0.0379 rpy=1.570796326795 0.0 0.0
- joint hand_r_mimic_distal_joint: axis -1.0 0.0 0.0 -> (none); origin xyz=0.0 0.0 0.07 -> (none)
- joint hand_r_proximal_joint: axis -1.0 0.0 0.0 -> (none); origin xyz=-0.01675 0.0245 -0.0175 rpy=0.0 0.0 0.0 -> (none)
- joint hand_r_spring_proximal_joint: axis -1.0 0.0 0.0 -> (none)
- joint head_center_camera_frame_joint: origin xyz=0.0195 0.0 0.061 rpy=-1.5707963268 0.0 -1.5707963268 -> (none)
- joint head_center_camera_gazebo_frame_joint: origin xyz=0 0 0 rpy=1.5707963268 -1.5707963268 0.0 -> xyz=0 0 0 rpy=1.570796326795 -1.570796326795 0.0
- joint head_l_stereo_camera_gazebo_frame_joint: origin xyz=0 0 0 rpy=1.5707963268 -1.5707963268 0.0 -> xyz=0 0 0 rpy=1.570796326795 -1.570796326795 0.0
- joint head_l_stereo_camera_joint: origin xyz=0.02 0.07 0.061 rpy=-1.5707963268 0.0 -1.5707963268 -> (none)
- joint head_pan_joint: origin xyz=0.0 0.0 0.0 rpy=0.0 0.0 0.0 -> (none)
- joint head_r_stereo_camera_gazebo_frame_joint: origin xyz=0 0 0 rpy=1.5707963268 -1.5707963268 0.0 -> xyz=0 0 0 rpy=1.570796326795 -1.570796326795 0.0
- joint head_r_stereo_camera_joint: origin xyz=0.02 -0.07 0.061 rpy=-1.5707963268 0.0 -1.5707963268 -> (none)
- joint head_rgbd_sensor_gazebo_frame_joint: origin xyz=0 0 0 rpy=1.5707963268 -1.5707963268 0.0 -> xyz=0 0 0 rpy=1.570796326795 -1.570796326795 0.0
- joint head_rgbd_sensor_joint: origin xyz=-0.079796 0.022 0.215172 rpy=-1.5707963268 0.0 -1.5707963268 -> (none)
- joint torso_lift_joint: origin xyz=0.0 0.0 0.752 rpy=0.0 0.0 0.0 -> (none)
- joint wrist_ft_sensor_frame_joint: origin xyz=0.0 0.0 0.0735 rpy=3.14159265359 0.0 0.0 -> (none)
